File: MaskRom-TSOP48-to-DIP42-adapter/MaskRom-TSOP48-to-DIP42-adapter.kicad_pcb (KiCad board)
At the start: 2 copper layers, 50 x 61 mm, 2 parts, among them J1 TSOP-48-breakout-board, U2 27C322

Commit message: next rev of tsop48-to-dip42
Routing:
- net /VSS: track 0.00 -> 84.2 mm, vias 0 -> 1
- net /D0: track 49.7 -> 28.0 mm
- net /D1: track 53.8 -> 35.2 mm
- net /~{OE}: track 50.3 -> 31.8 mm, vias 1 -> 0
- net /A18: track 47.1 -> 31.9 mm
- net /D3: track 40.7 -> 51.7 mm
- net /A15: track 44.2 -> 33.5 mm
- net /D2: track 31.0 -> 39.9 mm, vias 0 -> 1
- net /VCC: track 110.2 -> 101.7 mm
- net /D9: track 33.6 -> 41.0 mm
- net /A16: track 47.0 -> 39.7 mm
- net /A12: track 28.0 -> 35.1 mm
- net /A8: track 38.6 -> 45.1 mm
- net /D10: track 39.9 -> 45.4 mm
- net /D8: track 40.5 -> 35.2 mm
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- added copper zone on B.Cu, net /VSS
Other:
- board size 50 x 61 mm -> 50 x 54.7 mm
- board text added: "5V Mask ROM TSOP-48 -to- DIP-42 adapter v1.1"
- board text removed: "5V Mask ROM TSOP-48 -to- DIP-42 adapter v1"
